File: PCB/Schism PCB.kicad_sch (KiCad schematic)
At the start: 86 parts, among them J1 USB C Connector, J2 JTAG_TC2030, SW1 Boot, U1 XC6206, U2 USBLC6-2SC6, U3 RP2040, U4 W25Q128JVS, Y1 12MHz

Commit message: Final schematic and component placement
Parts:
- added MB5, MB6: MouseBites, PCM_marbastlib-various:mousebites_5p5mm_easysnap, symbol Mechanical:MountingHole
- added R1 (x4): 1M, Resistor_SMD:R_0603_1608Metric, symbol Device:R_Small
Connections:
- net A: now also J1.A7 (D-), J1.B7 (D-)
- net B: now also MX17.2, MX18.1
- net C_DN: now also J1.A10 (RX2-), J1.B10 (RX1-)
- net C_LT: now also J1.A6 (D+), J1.B6 (D+)
- net C_RT: now also J1.A11 (RX2+), J1.B11 (RX1+)
- net C_UP: now also J1.A2 (TX1+), J1.B2 (TX2+)
- net DOWN: now also J1.A6 (D+), J1.B6 (D+)
- net GND: now also J1.A1 (GND), J1.A1 (GND), J1.A1 (GND), J1.A1 (GND), J1.A12 (GND), J1.A12 (GND), J1.A12 (GND), J1.A12 (GND), J1.B1 (GND), J1.B1 (GND), J1.B1 (GND), J1.B1 (GND), J1.B12 (GND), J1.B12 (GND), J1.B12 (GND), J1.B12 (GND), MX1.2, MX10.1, MX11.1, MX12.2, MX13.2, MX14.1, MX15.1, MX16.2, MX17.1, MX18.2, MX19.1, MX2.1, MX20.2, MX21.2, MX22.1, MX23.1, MX24.2, MX25.1, MX26.2, MX27.1, MX28.2, MX29.1, MX3.2, MX30.2, MX31.1, MX32.2, MX33.1, MX34.2, MX35.2, MX36.1, MX37.2, MX38.1, MX39.2, MX4.1, MX40.1, MX41.2, MX42.1, MX5.1, MX6.2, MX7.1, MX8.2, MX9.2, R1.1, R1.1, R1.1, R1.1
- net L: now also J1.A8 (SBU1), J1.B8 (SBU2)
- net LEFT: now also J1.A7 (D-), J1.B7 (D-)
- net LS: now also MX29.2, MX30.1
- net M1: now also J1.A4 (VBUS), J1.A9 (VBUS), J1.B4 (VBUS), J1.B9 (VBUS)
- net M2: now also J1.A10 (RX2-), J1.B10 (RX1-)
- net MS: now also MX31.2, MX32.1
- net R: now also MX25.2, MX26.1
- net RIGHT: now also J1.A3 (TX1-), J1.B3 (TX2-)
- net START: now also J1.A2 (TX1+), J1.B2 (TX2+)
- net UP: now also MX23.2, MX24.1
- net X: now also MX19.2, MX20.1
- net Y: now also MX27.2, MX28.1
- net Z: now also MX21.1, MX22.2
- net M3: now reaches U3.11 (GPIO8)
- net M3: now also J1.A11 (RX2+), J1.B11 (RX1+)
- net C_RT_2: now reaches MX37.1, MX38.2
- net C_RT_2: now also J1.A11 (RX2+), J1.B11 (RX1+)
- net DOWN_2: now reaches MX5.2, MX6.1
- net DOWN_2: now also J1.A6 (D+), J1.B6 (D+)
- net M3_2: now reaches MX11.2, MX12.1
- net M3_2: now also J1.A11 (RX2+), J1.B11 (RX1+)
- net A_2: now reaches MX35.1, MX36.2
- net A_2: now also J1.A7 (D-), J1.B7 (D-)
- net M1_2: now reaches MX10.2, MX9.1
- net M1_2: now also J1.A4 (VBUS), J1.A9 (VBUS), J1.B4 (VBUS), J1.B9 (VBUS)
- net M2_2: now reaches MX13.1, MX14.2
- net M2_2: now also J1.A10 (RX2-), J1.B10 (RX1-)
- net C_LT_2: now reaches MX39.1, MX40.2
- net C_LT_2: now also J1.A6 (D+), J1.B6 (D+)
- net START_2: now reaches J1.A2 (TX1+)
- net START_2: now also J1.B2 (TX2+), MX15.2, MX16.1
- net RIGHT_2: now reaches J1.A3 (TX1-)
- net RIGHT_2: now also J1.B3 (TX2-), MX7.2, MX8.1
- net LEFT_2: now reaches J1.A7 (D-)
- net LEFT_2: now also J1.B7 (D-), MX3.1, MX4.2
- net L_2: now reaches J1.A8 (SBU1)
- net L_2: now also J1.B8 (SBU2), MX1.1, MX2.2
- net at J1.S1 (SHIELD): now also R1.2 (x4)
- net C_UP_2: now reaches MX41.1, MX42.2
- net C_UP_2: now also J1.A2 (TX1+), J1.B2 (TX2+)
- net C_DN_2: now reaches MX33.2, MX34.1
- net C_DN_2: now also J1.A10 (RX2-), J1.B10 (RX1-)
- no-connect marks 11 -> 28
Other:
- moved on the sheet: D2, D3, J1, MX1, MX10, MX11, MX12, MX13, MX14, MX15, MX16, MX17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

Commit message: v0.1
Parts:
- added H1, H2: qw-logo, qw-logo:qw new logo silk + copper sm, symbol Mechanical:MountingHole
- added H10, H11, H12, H7, H8, H9: 1999-logo, 1999:1999 logo md, symbol Mechanical:MountingHole
- added H3, H4, H5, H6: qw-logo, qw-logo:qw new logo silk + copper md, symbol Mechanical:MountingHole

Commit message: v0.1 choc version
Parts:
- MX1, MX12, MX13, MX16, MX18, MX20, MX21, MX24, MX26, MX28, MX3, MX30, MX32, MX34, MX35, MX37, MX39, MX41, MX6, MX8, MX9: footprint PCM_marbastlib-mx:SW_MX_HS_1u -> PCM_marbastlib-choc:SW_choc_v1_HS_1u
- MX10, MX11, MX14, MX15, MX17, MX19, MX2, MX22, MX23, MX25, MX27, MX29, MX31, MX33, MX36, MX38, MX4, MX40, MX42, MX5, MX7: footprint PCM_marbastlib-mx:SW_MX_1u -> PCM_marbastlib-choc:SW_choc_v1_1u

Commit message: Revert "v0.1 choc version"
This reverts commit 5703bf07c79f879200e349cafaf13ac2920e4a95.
Parts:
- MX1, MX12, MX13, MX16, MX18, MX20, MX21, MX24, MX26, MX28, MX3, MX30, MX32, MX34, MX35, MX37, MX39, MX41, MX6, MX8, MX9: footprint PCM_marbastlib-choc:SW_choc_v1_HS_1u -> PCM_marbastlib-mx:SW_MX_HS_1u
- MX10, MX11, MX14, MX15, MX17, MX19, MX2, MX22, MX23, MX25, MX27, MX29, MX31, MX33, MX36, MX38, MX4, MX40, MX42, MX5, MX7: footprint PCM_marbastlib-choc:SW_choc_v1_1u -> PCM_marbastlib-mx:SW_MX_1u

Commit message: v0.3 electrically connected
Parts:
- removed J1 (x4): USB C Connector, footprints:TYPE-C_24P_QCHT, symbol Connector:USB_C_Receptacle
- removed R1 (x4): 1M, Resistor_SMD:R_0603_1608Metric, symbol Device:R_Small
- added J3, J4: USB_C_Receptacle_USB2.0, PCM_marbastlib-various:USB_C_Receptacle_HRO_TYPE-C-31-M-12, symbol Connector:USB_C_Receptacle_USB2.0
- added J5, J6, J7: Conn_01x06_MountingPin, Connector_JST:JST_SH_SM06B-SRSS-TB_1x06-1MP_P1.00mm_Horizontal, symbol Connector_Generic_MountingPin:Conn_01x06_MountingPin
- added J8, J9: Conn_01x06, Connector_PinHeader_2.54mm:PinHeader_1x06_P2.54mm_Vertical, symbol Connector_Generic:Conn_01x06
- added R1 (x2): 1M, Resistor_SMD:R_0603_1608Metric, symbol Device:R_Small
- added U5: MCP23017_SO, Package_SO:SOIC-28W_7.5x17.9mm_P1.27mm, symbol Interface_Expansion:MCP23017_SO
Connections:
- net DOWN_2 is gone; now on net DOWN: MX5.2, MX6.1
- net LEFT_2 is gone; now on net LEFT: MX3.1, MX4.2
- net L_2 is gone; now on net L: MX1.1, MX2.2
- net M1_2 is gone; now on net M1: MX10.2, MX9.1
- net M2_2 is gone; now on net M2: MX13.1, MX14.2
- net M3_2 is gone; now on net M3: MX11.2, MX12.1
- net RIGHT_2 is gone; now on net RIGHT: MX7.2, MX8.1
- net START_2 is gone; now on net START: MX15.2, MX16.1
- net +3V3: now also J3.A4 (VBUS), J3.A9 (VBUS), J3.B4 (VBUS), J3.B9 (VBUS), J4.A4 (VBUS), J4.A9 (VBUS), J4.B4 (VBUS), J4.B9 (VBUS), U5.9 (VDD)
- net A: now also J5.3 (Pin_3), J8.3 (Pin_3), U5.4 (GPB3); no longer U3.17 (GPIO14)
- net A_2: now also J6.3 (Pin_3), J7.3 (Pin_3)
- net B: now also U5.28 (GPA7); no longer U3.38 (GPIO26/ADC0)
- net C_DN: now also J5.2 (Pin_2), J8.2 (Pin_2), U5.5 (GPB4); no longer U3.18 (GPIO15)
- net C_DN_2: now also J6.2 (Pin_2), J7.2 (Pin_2)
- net C_LT: now also J5.4 (Pin_4), J8.4 (Pin_4), U5.3 (GPB2); no longer U3.16 (GPIO13)
- net C_LT_2: now also J6.4 (Pin_4), J7.4 (Pin_4)
- net C_RT: now also J5.5 (Pin_5), J8.5 (Pin_5), U5.2 (GPB1); no longer U3.27 (GPIO16)
- net C_RT_2: now also J6.5 (Pin_5), J7.5 (Pin_5)
- net C_UP: now also J5.6 (Pin_6), J8.6 (Pin_6), U5.1 (GPB0); no longer U3.15 (GPIO12)
- net C_UP_2: now also J6.6 (Pin_6), J7.6 (Pin_6)
- net DOWN: now also U3.38 (GPIO26/ADC0); no longer U3.5 (GPIO3)
- net GND: now also J3.A1 (GND), J3.A12 (GND), J3.B1 (GND), J3.B12 (GND), J4.A1 (GND), J4.A12 (GND), J4.B1 (GND), J4.B12 (GND), J5.1 (Pin_1), J5.MP (MountPin), J6.1 (Pin_1), J6.MP (MountPin), J7.1 (Pin_1), J7.MP (MountPin), J8.1 (Pin_1), J9.1 (Pin_1), R1.1, R1.1, U5.10 (VSS)
- net L: now also U3.29 (GPIO18); no longer U3.7 (GPIO5)
- net LEFT: now also U3.30 (GPIO19); no longer U3.6 (GPIO4)
- net LS: now also U5.23 (GPA2); no longer U3.31 (GPIO20)
- net M1: now also U3.5 (GPIO3); no longer U3.8 (GPIO6)
- net M2: now also U3.4 (GPIO2); no longer U3.9 (GPIO7)
- net M3: now also U3.2 (GPIO0); no longer U3.11 (GPIO8)
- net MS: now also U5.25 (GPA4); no longer U3.29 (GPIO18)
- net R: now also U5.21 (GPA0); no longer U3.39 (GPIO27/ADC1)
- net RIGHT: now also U3.39 (GPIO27/ADC1); no longer U3.4 (GPIO2)
- net START: now also U3.3 (GPIO1); no longer U3.2 (GPIO0)
- net UP: now also U5.27 (GPA6); no longer U3.28 (GPIO17)
- net X: now also U5.24 (GPA3); no longer U3.32 (GPIO21)
- net Y: now also U5.22 (GPA1); no longer U3.34 (GPIO22)
- net Z: now also U5.26 (GPA5); no longer U3.30 (GPIO19)
- new net: J3.S1 (SHIELD), R1.2
- new net: J4.S1 (SHIELD), R1.2
- new net SCL: J3.A6 (D+), J3.B6 (D+), U3.32 (GPIO21)
- new net SCL_2: J4.A6 (D+), J4.B6 (D+), U5.12 (SCK)
- new net SDA: J3.A7 (D-), J3.B7 (D-), U3.31 (GPIO20)
- new net SDA_2: J4.A7 (D-), J4.B7 (D-), U5.13 (SDA)
- no-connect marks 28 -> 13

Commit message: Pre-production files v0.3
Parts:
- added C13: 100nF, Capacitor_SMD:C_0402_1005Metric, symbol Device:C_Small
- added J10: Conn_01x04_MountingPin, Connector_JST:JST_SH_SM04B-SRSS-TB_1x04-1MP_P1.00mm_Horizontal, symbol Connector_Generic_MountingPin:Conn_01x04_MountingPin
- added J11: USB_A, Connector_USB:USB_A_Receptacle_GCT_USB1046, symbol Connector:USB_A
- added J12: Conn_01x04, Connector_PinHeader_2.54mm:PinHeader_1x04_P2.54mm_Vertical, symbol Connector_Generic:Conn_01x04
- added J13: Conn_01x10, Connector_PinHeader_2.54mm:PinHeader_1x10_P2.54mm_Vertical, symbol Connector_Generic:Conn_01x10
- added R1: 1M, Resistor_SMD:R_0603_1608Metric, symbol Device:R_Small
- added R7 (x3): 10k, Resistor_SMD:R_0402_1005Metric, symbol Device:R_Small
- J5: value Conn_01x06_MountingPin -> JST
- J6: value Conn_01x06_MountingPin -> JST Left
- J7: value Conn_01x06_MountingPin -> JST Right
- J8: value Conn_01x06 -> 2.54 Header
- J9: value Conn_01x06 -> 2.54
Connections:
- net +3V3: now also C13.2, J10.1 (Pin_1), J11.1 (VBUS), J12.4 (Pin_4), R7.1, R7.2, R7.2
- net A_2: now also J6.5 (Pin_5), J7.5 (Pin_5), J9.3 (Pin_3); no longer J6.3 (Pin_3), J7.3 (Pin_3)
- net C_DN_2: now also J6.6 (Pin_6), J7.6 (Pin_6), J9.2 (Pin_2); no longer J6.2 (Pin_2), J7.2 (Pin_2)
- net C_LT_2: now also J9.4 (Pin_4)
- net C_RT_2: now also J6.3 (Pin_3), J7.3 (Pin_3), J9.5 (Pin_5); no longer J6.5 (Pin_5), J7.5 (Pin_5)
- net C_UP_2: now also J6.2 (Pin_2), J7.2 (Pin_2), J9.6 (Pin_6); no longer J6.6 (Pin_6), J7.6 (Pin_6)
- net GND: now also U5.15 (A0), U5.16 (A1), U5.17 (A2), C13.1, J10.4 (Pin_4), J10.MP (MountPin), J11.4 (GND), J12.1 (Pin_1), J13.1 (Pin_1), R1.1
- net MS: now also U5.26 (GPA5); no longer U5.25 (GPA4)
- net SCL_2: now also R7.1
- net SDA_2: now also R7.2
- net Z: now also U5.25 (GPA4); no longer U5.26 (GPA5)
- net EX5: now reaches U3.11 (GPIO8)
- net EX5: now also J13.6 (Pin_6)
- net EX4: now reaches U3.15 (GPIO12)
- net EX4: now also J13.5 (Pin_5)
- net EX3: now reaches U3.16 (GPIO13)
- net EX3: now also J13.4 (Pin_4)
- net EX2: now reaches U3.17 (GPIO14)
- net EX2: now also J13.3 (Pin_3)
- net EX1: now reaches U3.18 (GPIO15)
- net EX1: now also J13.2 (Pin_2)
- net PD+: now reaches U3.27 (GPIO16)
- net PD+: now also J10.3 (Pin_3), J11.3 (D+), J12.2 (Pin_2)
- net PD-: now reaches U3.28 (GPIO17)
- net PD-: now also J10.2 (Pin_2), J11.2 (D-), J12.3 (Pin_3)
- net EX9: now reaches U3.6 (GPIO4)
- net EX9: now also J13.10 (Pin_10)
- net EX8: now reaches U3.7 (GPIO5)
- net EX8: now also J13.9 (Pin_9)
- net EX7: now reaches U3.8 (GPIO6)
- net EX7: now also J13.8 (Pin_8)
- net EX6: now reaches U3.9 (GPIO7)
- net EX6: now also J13.7 (Pin_7)
- net at U5.18 (~{RESET}): now also R7.1
- new net: J11.5 (Shield), R1.2
- no-connect marks 13 -> 18
Other:
- note added: "Buttons"
- note added: "C PAD"
- note added: "Connectors"
- note added: "LEFT HAND"
- note added: "Logos and Mousebites"
- note added: "RIGHT HAND"
- note added: "USB C i2c port"
- note added: "i2c chip"
- moved on the sheet: D2, D3, J3, J4, J5, J6, J7, J8, J9, MB5, MB6, MX1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

Commit message: v0.5
Parts:
- removed U5: MCP23017_SO, Package_SO:SOIC-28W_7.5x17.9mm_P1.27mm, symbol Interface_Expansion:MCP23017_SO
- added U6: PCA9671PW_118, TSSOP24_SOT355-1_NXP, symbol PCA9671PW:PCA9671PW_118
- J10, J11, J13, MB5, MB6: now left out of the parts list
- J3, J4: LCSC (none) -> C165948
- J5, J6, J7: LCSC (none) -> C160405
Connections:
- net +3V3: now also U6.24 (VDD)
- net A: now also J5.2 (Pin_2), U6.19 (P16); no longer J5.3 (Pin_3)
- net B: now also U6.11 (P07)
- net C_DN: now also J5.1 (Pin_1), U6.20 (P17); no longer J5.2 (Pin_2)
- net C_LT: now also J5.3 (Pin_3), U6.18 (P15); no longer J5.4 (Pin_4)
- net C_RT: now also J5.4 (Pin_4), U6.17 (P14); no longer J5.5 (Pin_5)
- net C_UP: now also J5.5 (Pin_5), U6.16 (P13); no longer J5.6 (Pin_6)
- net GND: now also J5.6 (Pin_6), U6.12 (VSS), U6.2 (AD1), U6.21 (AD0), U6.3 (AD2); no longer J5.1 (Pin_1)
- net LS: now also U6.6 (P02)
- net MS: now also U6.9 (P05)
- net R: now also U6.4 (P00)
- net SCL_2: now also U6.22 (SCL)
- net SDA_2: now also U6.23 (SDA)
- net UP: now also U6.10 (P06)
- net X: now also U6.7 (P03)
- net Y: now also U6.5 (P01)
- net Z: now also U6.8 (P04)
- net at R7.1: now also U6.1 (*RESET)
- no-connect marks 18 -> 19
Other:
- moved on the sheet: C13, R7
